Commit message: changed planar robot appearance

File: mushroom_rl/environments/pybullet_envs/data/air_hockey/planar/planar_robot_1.urdf (robot description, URDF)
Before this commit: robot planar_robot_1, 7 links, 6 joints
Links:
- link planar_robot_1/link_1: geometry collision cylinder length=0.5 radius=0.04; visual cylinder length=0.5 radius=0.04
- link planar_robot_1/link_2: geometry collision cylinder length=0.4 radius=0.04; visual cylinder length=0.4 radius=0.04
- link planar_robot_1/link_3: geometry collision cylinder length=0.4 radius=0.04; visual cylinder length=0.4 radius=0.04
