Commit message: changed color of robot

File: mushroom_rl/environments/pybullet_envs/data/air_hockey/planar/planar_robot_2.urdf (robot description, URDF)
Before this commit: robot planar_robot_2, 7 links, 6 joints
Links:
- removed link planar_robot_2/base_link
- removed link planar_robot_2/link_1
- removed link planar_robot_2/link_2
- removed link planar_robot_2/link_3
- removed link planar_robot_2/link_striker_ee
- removed link planar_robot_2/link_striker_hand
- added link planar_robot_1/base_link, mass 1; collision cylinder length=0.4 radius=0.075; visual cylinder length=0.4 radius=0.075
- added link planar_robot_1/link_1, mass 3; collision cylinder length=0.5 radius=0.04; visual cylinder length=0.5 radius=0.04
- added link planar_robot_1/link_2, mass 2.4; collision cylinder length=0.4 radius=0.04; visual cylinder length=0.4 radius=0.04
- added link planar_robot_1/link_3, mass 2.4; collision cylinder length=0.4 radius=0.04; visual cylinder length=0.4 radius=0.04
- added link planar_robot_1/link_striker_ee, mass 0.1; collision cylinder length=0.1 radius=0.05; visual cylinder length=0.02 radius=0.05
- added link planar_robot_1/link_striker_hand, mass 0.1; collision cylinder length=0.189 radius=0.01; visual cylinder length=0.189 radius=0.01
Joints:
- removed joint planar_robot_2/base_joint
- removed joint planar_robot_2/joint_1
- removed joint planar_robot_2/joint_2
- removed joint planar_robot_2/joint_3
- removed joint planar_robot_2/joint_striker
- removed joint planar_robot_2/joint_striker_ee
- added joint planar_robot_1/base_joint: type fixed, parent world, child planar_robot_1/base_link, origin xyz=0.0 0.0 0.0 rpy=0.0 0.0 0.0
- added joint planar_robot_1/joint_1: type revolute, parent planar_robot_1/base_link, child planar_robot_1/link_1, origin xyz=0.0 0.0 0.0 rpy=0.0 0.0 0.0, axis 0 0 1, limit lower=-2.9670597283903604 upper=2.9670597283903604 effort=40.0 velocity=2.35619449019
- added joint planar_robot_1/joint_2: type revolute, parent planar_robot_1/link_1, child planar_robot_1/link_2, origin xyz=0.5 0 0, axis 0 0 1, limit lower=-2.0943951023931953 upper=2.0943951023931953 effort=15.0 velocity=2.35619449019
- added joint planar_robot_1/joint_3: type revolute, parent planar_robot_1/link_2, child planar_robot_1/link_3, origin xyz=0.4 0 0, axis 0 0 1, limit lower=-2.0943951023931953 upper=2.0943951023931953 effort=2.0 velocity=2.35619449019
- added joint planar_robot_1/joint_striker: type fixed, parent planar_robot_1/link_3, child planar_robot_1/link_striker_hand, origin xyz=0.4 0 0.0, axis 1 0 0
- added joint planar_robot_1/joint_striker_ee: type fixed, parent planar_robot_1/link_striker_hand, child planar_robot_1/link_striker_ee, origin xyz=0.0 0 -0.189, axis 1 0 0
